Commit message: add jsk_fetch.urdf.xacro in jsk_fetch_startup

File: jsk_fetch_robot/jsk_fetch_startup/robots/jsk_fetch.urdf.xacro (robot description, xacro)
@@ -2,9 +2,17 @@
 <robot name="fetch" xmlns:xacro="http://www.ros.org/wiki/xacro">
   <xacro:include filename="/etc/ros/indigo/calibrated_latest.urdf" />
+  <link name="t265_base_link">
+  </link>
+  <joint name="t265_to_base_virtual_joint" type="fixed">
+    <origin rpy="0 0 0" xyz="0 0 0" />
+    <parent link="t265_base_link" />
+    <child link="base_link" />
+    <axis xyz="0 0 1" />
+  </joint>
   <link name="base_camera_mount">
     <inertial>
-      <origin rpy="0 0.523598775 0" xyz="0 0 0" />
-      <mass value="0.17" />
-      <inertia ixx="0.024" ixy="0.01" ixz="0.034" iyy="0.034" iyz="0.024" izz="0.01" />
+      <origin rpy="0 0 0" xyz="0 0 0" />
+      <mass value="70.1294" />
+      <inertia ixx="1.225" ixy="0.0099" ixz="0.0062" iyy="1.2853" iyz="-0.0034" izz="0.987" />
     </inertial>
     <visual>

Commit message: changed parameters and link names of jsk_fetch.urdf.xacro

File: jsk_fetch_robot/jsk_fetch_startup/robots/jsk_fetch.urdf.xacro (robot description, xacro)
@@ -2,9 +2,9 @@
 <robot name="fetch" xmlns:xacro="http://www.ros.org/wiki/xacro">
   <xacro:include filename="/etc/ros/indigo/calibrated_latest.urdf" />
-  <link name="t265_base_link">
+  <link name="t265_pose_frame">
   </link>
   <joint name="t265_to_base_virtual_joint" type="fixed">
-    <origin rpy="0 0 0" xyz="0 0 0" />
-    <parent link="t265_base_link" />
+    <origin rpy="0 0 0" xyz="0.270 0.0081 0.4152" />
+    <parent link="t265_pose_frame" />
     <child link="base_link" />
     <axis xyz="0 0 1" />
@@ -12,7 +12,7 @@
   <link name="base_camera_mount">
     <inertial>
-      <origin rpy="0 0 0" xyz="0 0 0" />
-      <mass value="70.1294" />
-      <inertia ixx="1.225" ixy="0.0099" ixz="0.0062" iyy="1.2853" iyz="-0.0034" izz="0.987" />
+      <origin rpy="0 0.523598775 0" xyz="0 0 0" />
+      <mass value="0.17" />
+      <inertia ixx="0.024" ixy="0.01" ixz="0.034" iyy="0.034" iyz="0.024" izz="0.01" />
     </inertial>
     <visual>

Commit message: delete a t265 link

File: jsk_fetch_robot/jsk_fetch_startup/robots/jsk_fetch.urdf.xacro (robot description, xacro)
@@ -2,12 +2,4 @@
 <robot name="fetch" xmlns:xacro="http://www.ros.org/wiki/xacro">
   <xacro:include filename="/etc/ros/indigo/calibrated_latest.urdf" />
-  <link name="t265_pose_frame">
-  </link>
-  <joint name="t265_to_base_virtual_joint" type="fixed">
-    <origin rpy="0 0 0" xyz="0.270 0.0081 0.4152" />
-    <parent link="t265_pose_frame" />
-    <child link="base_link" />
-    <axis xyz="0 0 1" />
-  </joint>
   <link name="base_camera_mount">
     <inertial>

Commit message: [jsk_fetch_startup] add a fetch head box link to xacro

File: jsk_fetch_robot/jsk_fetch_startup/robots/jsk_fetch.urdf.xacro (robot description, xacro)
@@ -38,3 +38,30 @@
     <axis xyz="0 0 1" />
   </joint>
+  <joint name="head_box_virtual_joint" type="fixed">
+    <origin rpy="0 0 0" xyz="0 0 0" />
+    <parent link="head_pan_link" />
+    <child link="head_box_link" />
+  </joint>
+  <link name="head_box_link" >
+    <inertial>
+      <origin rpy="0 0 0" xyz="0 0 0" />
+      <mass value="1" />
+      <inertial ixx="1" ixy="0" ixz="0" iyy="1" iyz="0" izz="1" />
+    </inertial>
+    <visual>
+      <origin rpy="0 0 0" xyz="0 0 0" />
+      <geometry>
+        <mesh filename="package://jsk_fetch_accessories/head_box/fetch_head_box_simplified.stl" scale="0.001 0.001 0.001" />
+      </geometry>
+      <material name="">
+        <color rgba="0.356 0.361 0.376 1" />
+      </material>
+    </visual>
+    <collision>
+      <origin rpy="0 0 0" xyz="0 0 0" />
+      <geometry>
+        <mesh filename="package://jsk_fetch_accessories/head_box/fetch_head_box_simplified.stl" scale="0.001 0.001 0.001" />
+      </geometry>
+    </collision>
+  </link>
 </robot>

Commit message: [jsk_fetch_startup] fix head box name

File: jsk_fetch_robot/jsk_fetch_startup/robots/jsk_fetch.urdf.xacro (robot description, xacro)
@@ -44,5 +44,5 @@
       <origin rpy="0 0 0" xyz="0 0 0" />
       <geometry>
-        <mesh filename="package://jsk_fetch_accessories/head_box/fetch_head_box_simplified.stl" scale="0.001 0.001 0.001" />
+        <mesh filename="package://jsk_fetch_accessories/head_box/fetch_head_box_v2_simplified.stl" scale="0.001 0.001 0.001" />
       </geometry>
       <material name="">
@@ -53,5 +53,5 @@
       <origin rpy="0 0 0" xyz="0 0 0" />
       <geometry>
-        <mesh filename="package://jsk_fetch_accessories/head_box/fetch_head_box_simplified.stl" scale="0.001 0.001 0.001" />
+        <mesh filename="package://jsk_fetch_accessories/head_box/fetch_head_box_v2_simplified.stl" scale="0.001 0.001 0.001" />
       </geometry>
     </collision>

Commit message: fix typo in jsk_fetch.urdf.xacro

File: jsk_fetch_robot/jsk_fetch_startup/robots/jsk_fetch.urdf.xacro (robot description, xacro)
@@ -39,5 +39,5 @@
       <origin rpy="0 0 0" xyz="0 0 0" />
       <mass value="1" />
-      <inertial ixx="1" ixy="0" ixz="0" iyy="1" iyz="0" izz="1" />
+      <inertia ixx="1" ixy="0" ixz="0" iyy="1" iyz="0" izz="1" />
     </inertial>
     <visual>

Commit message: make base_camera_mount and head_box xacro

File: jsk_fetch_robot/jsk_fetch_startup/robots/jsk_fetch.urdf.xacro (robot description, xacro)
@@ -1,59 +1,12 @@
 <?xml version="1.0" ?>
 <robot name="fetch" xmlns:xacro="http://www.ros.org/wiki/xacro">
+  <xacro:arg name="base_camera_mount" default="true" />
+  <xacro:arg name="head_box" default="true" />
   <xacro:include filename="/etc/ros/indigo/calibrated_latest.urdf" />
-  <link name="base_camera_mount">
-    <inertial>
-      <origin rpy="0 0.523598775 0" xyz="0 0 0" />
-      <mass value="0.17" />
-      <inertia ixx="0.024" ixy="0.01" ixz="0.034" iyy="0.034" iyz="0.024" izz="0.01" />
-    </inertial>
-    <visual>
-      <origin rpy="0 0 0" xyz="0 0 0" />
-      <geometry>
-        <mesh filename="package://jsk_fetch_accessories/base_camera_mount_mk1/fetch_base_camera_mount_mk1_main.stl" scale="0.001 0.001 0.001" />
-      </geometry>
-      <material name="">
-        <color rgba="0.356 0.361 0.376 1" />
-      </material>
-    </visual>
-    <collision>
-      <origin rpy="0 0 0" xyz="0 0 0" />
-      <geometry>
-        <mesh filename="package://jsk_fetch_accessories/base_camera_mount_mk1/fetch_base_camera_mount_mk1_collision.stl" scale="0.001 0.001 0.001" />
-      </geometry>
-    </collision>
-  </link>
-  <joint name="base_camera_mount_joint" type="fixed">
-    <origin rpy="0 0 0" xyz="0 0 0" />
-    <parent link="base_link" />
-    <child link="base_camera_mount" />
-    <axis xyz="0 0 1" />
-  </joint>
-  <joint name="head_box_virtual_joint" type="fixed">
-    <origin rpy="0 0 0" xyz="0 0 0" />
-    <parent link="head_pan_link" />
-    <child link="head_box_link" />
-  </joint>
-  <link name="head_box_link" >
-    <inertial>
-      <origin rpy="0 0 0" xyz="0 0 0" />
-      <mass value="1" />
-      <inertia ixx="1" ixy="0" ixz="0" iyy="1" iyz="0" izz="1" />
-    </inertial>
-    <visual>
-      <origin rpy="0 0 0" xyz="0 0 0" />
-      <geometry>
-        <mesh filename="package://jsk_fetch_accessories/head_box/fetch_head_box_v2_simplified.stl" scale="0.001 0.001 0.001" />
-      </geometry>
-      <material name="">
-        <color rgba="0.356 0.361 0.376 1" />
-      </material>
-    </visual>
-    <collision>
-      <origin rpy="0 0 0" xyz="0 0 0" />
-      <geometry>
-        <mesh filename="package://jsk_fetch_accessories/head_box/fetch_head_box_v2_simplified.stl" scale="0.001 0.001 0.001" />
-      </geometry>
-    </collision>
-  </link>
+  <xacro:if value="$(arg base_camera_mount)">
+    <xacro:include filename="$(find jsk_fetch_startup)/robots/base_camera_mount.urdf.xacro" />
+  </xacro:if>
+  <xacro:if value="$(arg head_box)">
+    <xacro:include filename="$(find jsk_fetch_startup)/robots/head_box.urdf.xacro" />
+  </xacro:if>
 </robot>
