Commit message: [jsk_fetch_accessories][jsk_fetch_startup] add fetch_base_camera_mount_mk2 and make it a default

File: jsk_fetch_robot/jsk_fetch_startup/robots/base_camera_mount.urdf.xacro (robot description, xacro)
@@ -1,31 +1,66 @@
 <?xml version="1.0" ?>
 <robot name="base_camera_mount" xmlns:xacro="http://www.ros.org/wiki/xacro">
-  <link name="base_camera_mount">
-    <inertial>
-      <origin rpy="0 0.523598775 0" xyz="0 0 0" />
-      <mass value="0.17" />
-      <inertia ixx="0.024" ixy="0.01" ixz="0.034" iyy="0.034" iyz="0.024" izz="0.01" />
-    </inertial>
-    <visual>
-      <origin rpy="0 0 0" xyz="0 0 0" />
-      <geometry>
-        <mesh filename="package://jsk_fetch_accessories/base_camera_mount_mk1/fetch_base_camera_mount_mk1_main.stl" scale="0.001 0.001 0.001" />
-      </geometry>
-      <material name="">
-        <color rgba="0.356 0.361 0.376 1" />
-      </material>
-    </visual>
-    <collision>
-      <origin rpy="0 0 0" xyz="0 0 0" />
-      <geometry>
-        <mesh filename="package://jsk_fetch_accessories/base_camera_mount_mk1/fetch_base_camera_mount_mk1_collision.stl" scale="0.001 0.001 0.001" />
-      </geometry>
-    </collision>
-  </link>
-  <joint name="base_camera_mount_joint" type="fixed">
-    <origin rpy="0 0 0" xyz="0 0 0" />
-    <parent link="base_link" />
-    <child link="base_camera_mount" />
-    <axis xyz="0 0 1" />
-  </joint>
+  <xacro:arg name="version" default="2" />
+  <!-- mk1 -->
+  <xacro:if value="${version == '1'}">
+      <link name="base_camera_mount">
+        <inertial>
+          <origin rpy="0 0.523598775 0" xyz="0 0 0" />
+          <mass value="0.17" />
+          <inertia ixx="0.024" ixy="0.01" ixz="0.034" iyy="0.034" iyz="0.024" izz="0.01" />
+        </inertial>
+        <visual>
+          <origin rpy="0 0 0" xyz="0 0 0" />
+          <geometry>
+            <mesh filename="package://jsk_fetch_accessories/base_camera_mount_mk1/fetch_base_camera_mount_mk1_main.stl" scale="0.001 0.001 0.001" />
+          </geometry>
+          <material name="">
+            <color rgba="0.356 0.361 0.376 1" />
+          </material>
+        </visual>
+        <collision>
+          <origin rpy="0 0 0" xyz="0 0 0" />
+          <geometry>
+            <mesh filename="package://jsk_fetch_accessories/base_camera_mount_mk1/fetch_base_camera_mount_mk1_collision.stl" scale="0.001 0.001 0.001" />
+          </geometry>
+        </collision>
+      </link>
+      <joint name="base_camera_mount_joint" type="fixed">
+        <origin rpy="0 0 0" xyz="0 0 0" />
+        <parent link="base_link" />
+        <child link="base_camera_mount" />
+        <axis xyz="0 0 1" />
+      </joint>
+  </xacro:if>
+  <!-- mk2 -->
+  <xacro:if value="${version == '2'}">
+      <link name="base_camera_mount">
+          <inertial>
+              <origin rpy="0 0 0" xyz="0 0 0" />
+              <mass value="0" />
+              <inertia ixx="0" ixy="0" ixz="0" iyy="0" iyz="0" izz="0" />
+          </inertial>
+          <visual>
+              <origin rpy="0 0 0" xyz="0 0 0" />
+              <geometry>
+                  <mesh filename="package://jsk_fetch_accessories/base_camera_mount_mk2/fetch_base_camera_mount_mk2_main.stl" scale="0.001 0.001 0.001" />
+              </geometry>
+              <material name="">
+                <color rgba="0.356 0.361 0.376 1" />
+              </material>
+          </visual>
+          <collision>
+              <origin rpy="0 0 0" xyz="0 0 0" />
+              <geometry>
+                  <mesh filename="package://jsk_fetch_accessories/base_camera_mount_mk2/fetch_base_camera_mount_mk2_collision.stl" scale="0.001 0.001 0.001" />
+              </geometry>
+          </collision>
+      </link>
+      <joint name="base_camera_mount_joint" type="fixed">
+        <origin rpy="0 0 0" xyz="0 0 0" />
+        <parent link="base_link" />
+        <child link="base_camera_mount" />
+        <axis xyz="0 0 1" />
+      </joint>
+    </xacro:if>
 </robot>

Commit message: [jsk_fetch_startup] update link and joint parameters

File: jsk_fetch_robot/jsk_fetch_startup/robots/base_camera_mount.urdf.xacro (robot description, xacro)
@@ -63,4 +63,18 @@
         <axis xyz="0 0 1" />
       </joint>
+      <link name="d435_front_right_link" type="fixed" />
+      <joint name="base_link_to_d435_front_right_virtual_joint" >
+        <origin rpy="0 0.524 -0.524" xyz="0.242 -0.14 0.375" />
+        <parent link="base_link" />
+        <child link="d435_front_right_link" />
+        <axis xyz="0 0 1" />
+      </joint>
+      <link name="d435_front_left_link" type="fixed" />
+      <joint name="base_link_to_d435_front_left_virtual_joint" >
+        <origin rpy="0 0.524 0.524" xyz="0.242 0.14 0.375" />
+        <parent link="base_link" />
+        <child link="d435_front_left_link" />
+        <axis xyz="0 0 1" />
+      </joint>
     </xacro:if>
 </robot>

Commit message: [jsk_fetch_startup] fix bugs in xacro

File: jsk_fetch_robot/jsk_fetch_startup/robots/base_camera_mount.urdf.xacro (robot description, xacro)
@@ -3,5 +3,5 @@
   <xacro:arg name="version" default="2" />
   <!-- mk1 -->
-  <xacro:if value="${version == '1'}">
+  <xacro:if value="${$(arg version) == 1}">
       <link name="base_camera_mount">
         <inertial>
@@ -34,5 +34,5 @@
   </xacro:if>
   <!-- mk2 -->
-  <xacro:if value="${version == '2'}">
+  <xacro:if value="${$(arg version) == 2}">
       <link name="base_camera_mount">
           <inertial>
@@ -63,6 +63,6 @@
         <axis xyz="0 0 1" />
       </joint>
-      <link name="d435_front_right_link" type="fixed" />
-      <joint name="base_link_to_d435_front_right_virtual_joint" >
+      <link name="d435_front_right_link" />
+      <joint name="base_link_to_d435_front_right_virtual_joint" type="fixed" >
         <origin rpy="0 0.524 -0.524" xyz="0.242 -0.14 0.375" />
         <parent link="base_link" />
@@ -70,6 +70,6 @@
         <axis xyz="0 0 1" />
       </joint>
-      <link name="d435_front_left_link" type="fixed" />
-      <joint name="base_link_to_d435_front_left_virtual_joint" >
+      <link name="d435_front_left_link" />
+      <joint name="base_link_to_d435_front_left_virtual_joint" type="fixed" >
         <origin rpy="0 0.524 0.524" xyz="0.242 0.14 0.375" />
         <parent link="base_link" />
