Commit message: [jsk_unitree_description] add base_footprint link

File: jsk_unitree_robot/jsk_unitree_description/xacro/jsk_go1.xacro (robot description, xacro)
@@ -5,8 +5,14 @@
     <xacro:include filename="$(find go1_description)/xacro/robot.xacro">
     </xacro:include>
+    <link name="base_footprint"/>
+    <joint name="base_static_joint" type="fixed">
+        <origin rpy="0 0 0" xyz="0 0 -0.3"/>
+        <parent link="trunk"/>
+        <child link="base_footprint"/>
+    </joint>
     <!-- realsense mount -->
     <xacro:if value="$(arg use_realsense)">
         <link name="d435_top_link"/>
-        <joint name="base_static_joint" type="fixed">
+        <joint name="d435_top_joint" type="fixed">
             <origin rpy="0 0 0" xyz="0.120 0 0.115"/>
             <parent link="trunk"/>

Commit message: [jsk_unitree_description] add t265 and laser

File: jsk_unitree_robot/jsk_unitree_description/xacro/jsk_go1.xacro (robot description, xacro)
@@ -19,4 +19,16 @@
             <child link="d435_top_link"/>
         </joint>
+        <link name="t265_link"/>
+        <joint name="t265_joint" type="fixed">
+            <origin rpy="0 0 0" xyz="-0.120 0 -0.145"/>
+            <parent link="t265_link"/>
+            <child link="base"/>
+        </joint>
+        <link name="laser"/>
+        <joint name="d435_top_joint" type="fixed">
+            <origin rpy="0 0 0" xyz="-0.08 0 0.05"/>
+            <parent link="d435_top_link"/>
+            <child link="laser"/>
+        </joint>
     </xacro:if>
 </robot>

Commit message: [jsk_unitree_startup][jsk_unitree_description] update

File: jsk_unitree_robot/jsk_unitree_description/xacro/jsk_go1.xacro (robot description, xacro)
@@ -26,5 +26,5 @@
         </joint>
         <link name="laser"/>
-        <joint name="d435_top_joint" type="fixed">
+        <joint name="laser_joint" type="fixed">
             <origin rpy="0 0 0" xyz="-0.08 0 0.05"/>
             <parent link="d435_top_link"/>

Commit message: [jsk_unitree_description] fix xacro

File: jsk_unitree_robot/jsk_unitree_description/xacro/jsk_go1.xacro (robot description, xacro)
@@ -1,5 +1,5 @@
 <?xml version="1.0"?>
 <robot name="go1_description" xmlns:xacro="http://www.ros.org/wiki/xacro">
-    <xacro:arg name="use_realsense" default="true"/>
+    <xacro:arg name="use_navigation_unit" default="true"/>
     <xacro:arg name="DEBUG" default="false" />
     <xacro:include filename="$(find go1_description)/xacro/robot.xacro">
@@ -7,10 +7,10 @@
     <link name="base_footprint"/>
     <joint name="base_static_joint" type="fixed">
-        <origin rpy="0 0 0" xyz="0 0 -0.3"/>
-        <parent link="trunk"/>
-        <child link="base_footprint"/>
+        <origin rpy="0 0 0" xyz="0 0 0.3"/>
+        <parent link="base_footprint"/>
+        <child link="base"/>
     </joint>
     <!-- realsense mount -->
-    <xacro:if value="$(arg use_realsense)">
+    <xacro:if value="$(arg use_navigation_unit)">
         <link name="d435_top_link"/>
         <joint name="d435_top_joint" type="fixed">
@@ -18,10 +18,4 @@
             <parent link="trunk"/>
             <child link="d435_top_link"/>
-        </joint>
-        <link name="t265_link"/>
-        <joint name="t265_joint" type="fixed">
-            <origin rpy="0 0 0" xyz="-0.120 0 -0.145"/>
-            <parent link="t265_link"/>
-            <child link="base"/>
         </joint>
         <link name="laser"/>
